File: Hardware/Domofon.sch (EAGLE design)
At the start: 82 parts, among them J3 USB_A_PTH_MALE, Q1 BC817-40SMD, Q2 BC817-40SMD, Q3 BC817-40SMD, Q4 BC817-40SMD, Q5 SS8050-G, Q6 SS8050-G, U1 IP5306, U2 ESP-WROOM-32EU, U3 AMS1117, U4 CH340K, U5 PAM8403

Commit message: Защита от скачков по USB
Parts:
- added D7, D8, D9: 5.6V, SparkFun-DiscreteSemi:DIODE-ZENER-MMSZ5232BS
- added F1, F2: 16V/2.5A(5A TRIP), SparkFun-Fuses:PPTC_16V_2.5A
- added U6: AZC099-04S, SamacSys_Parts:AZC099-04S
Connections:
- new net N$43: F1.1, J3.VBUS
- new net N$44: BT2.POS, F2.2
- net 3.3V: now also D7.C
- net 5V: now also D8.C
- net GND: now also D7.A, D8.A, D9.A, U6.GND
- net N$19: now also D9.C, F2.1; no longer BT2.POS
- net N$5: now also F1.2, U6.VDD; no longer J3.VBUS
- net USBU_DM: now also U6.IO1
- net USBU_DP: now also U6.IO2
Other:
- moved on the sheet: BT2
